File: _autosave-stm32_board.kicad_pcb (KiCad board)
At the start: 2 copper layers, 28 parts, among them J1 USB_B_Micro, J2 Conn_01x04_Pin, J3 Conn_01x04_Pin, J4 Conn_01x04_Pin, SW1 SW_SPDT, U1 AMS1117-3.3, U2 STM32F103C8Tx, Y1 16MHz

Commit message: Updated PCB and added step file
Parts:
- SW1: footprint Button_Switch_THT:SW_E-Switch_EG1224_SPDT_Angled -> Button_Switch_SMD:SW_SPDT_PCM12
Changed lines of the file:
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@@
     )
   )
-  (footprint "Button_Switch_THT:SW_E-Switch_EG1224_SPDT_Angled" (layer "F.Cu")
+  (footprint "Button_Switch_SMD:SW_SPDT_PCM12" (layer "F.Cu")
     (at 147.69 107.745)
-    (descr "E-Switch slide switch, EG series, SPDT, right angle, http://spec_sheets.e-switch.com/specs/P040042.pdf")
-    (tags "switch SPDT")
+    (descr "Ultraminiature Surface Mount Slide Switch, right-angle, https://www.ckswitches.com/media/1424/pcm.pdf")
     (property "Sheetfile" "stm32_board.kicad_sch")
     (property "Sheetname" "")
     (property "ki_description" "Switch, single pole double throw")
     (property "ki_keywords" "switch single-pole double-throw spdt ON-ON")
-    (attr through_hole)
-    (fp_text reference "SW1" (at 4 -2.95) (layer "F.SilkS")
+    (attr smd)
+    (fp_text reference "SW1" (at 0 -3.2) (layer "F.SilkS")
         (effects (font (size 1 1) (thickness 0.15)))
     )
-    (fp_text value "SW_SPDT" (at 4 14.45) (layer "F.Fab")
+    (fp_text value "SW_SPDT" (at 0 4.25) (layer "F.Fab")
         (effects (font (size 1 1) (thickness 0.15)))
     )
-    (fp_text user "${REFERENCE}" (at 4 1.25) (layer "F.Fab")
-        (effects (font (size 1 1) (thickness 0.1)))
+    (fp_text user "${REFERENCE}" (at 0 -3.2) (layer "F.Fab")
+        (effects (font (size 1 1) (thickness 0.15)))
     )
-    (fp_line (start -3.3 -3.05) (end -2 -3.05)
+    (fp_line (start -3.45 -0.07) (end -3.45 0.72)
       (stroke (width 0.12) (type solid)) (layer "F.SilkS"))
-    (fp_line (start -3.3 -1.75) (end -3.3 -3.05)
+    (fp_line (start -2.85 1.73) (end 2.85 1.73)
       (stroke (width 0.12) (type solid)) (layer "F.SilkS"))
-    (fp_line (start -3 3.85) (end -3 -1.35)
+    (fp_line (start -1.6 -1.12) (end 0.1 -1.12)
       (stroke (width 0.12) (type solid)) (layer "F.SilkS"))
-    (fp_line (start -0.95 -2.1) (end 8.95 -2.1)
+    (fp_line (start -1.4 1.73) (end -1.4 3.02)
       (stroke (width 0.12) (type solid)) (layer "F.SilkS"))
-    (fp_line (start 8.95 4.6) (end -0.95 4.6)
+    (fp_line (start -1.4 3.02) (end -1.2 3.23)
       (stroke (width 0.12) (type solid)) (layer "F.SilkS"))
-    (fp_line (start 11 -1.35) (end 11 3.85)
+    (fp_line (start -1.2 3.23) (end -0.3 3.23)
       (stroke (width 0.12) (type solid)) (layer "F.SilkS"))
-    (fp_line (start -3.25 -3) (end 11.25 -3)
+    (fp_line (start -0.1 3.02) (end -0.3 3.23)
+      (stroke (width 0.12) (type solid)) (layer "F.SilkS"))
+    (fp_line (start -0.1 3.02) (end -0.1 1.73)
+      (stroke (width 0.12) (type solid)) (layer "F.SilkS"))
+    (fp_line (start 1.4 -1.12) (end 1.6 -1.12)
+      (stroke (width 0.12) (type solid)) (layer "F.SilkS"))
+    (fp_line (start 3.45 0.72) (end 3.45 -0.07)
+      (stroke (width 0.12) (type solid)) (layer "F.SilkS"))
+    (fp_line (start -4.4 -2.45) (end 4.4 -2.45)
       (stroke (width 0.05) (type solid)) (layer "F.CrtYd"))
-    (fp_line (start -3.25 5.5) (end -3.25 -3)
+    (fp_line (start -4.4 2.1) (end -4.4 -2.45)
       (stroke (width 0.05) (type solid)) (layer "F.CrtYd"))
-    (fp_line (start -0.75 5.5) (end -3.25 5.5)
+    (fp_line (start -1.65 2.1) (end -4.4 2.1)
       (stroke (width 0.05) (type solid)) (layer "F.CrtYd"))
-    (fp_line (start -0.75 13.75) (end -0.75 5.5)
+    (fp_line (start -1.65 3.4) (end -1.65 2.1)
       (stroke (width 0.05) (type solid)) (layer "F.CrtYd"))
-    (fp_line (start 8.75 5.5) (end 8.75 13.75)
+    (fp_line (start 1.65 2.1) (end 1.65 3.4)
       (stroke (width 0.05) (type solid)) (layer "F.CrtYd"))
-    (fp_line (start 8.75 13.75) (end -0.75 13.75)
+    (fp_line (start 1.65 3.4) (end -1.65 3.4)
       (stroke (width 0.05) (type solid)) (layer "F.CrtYd"))
-    (fp_line (start 11.25 -3) (end 11.25 5.5)
+    (fp_line (start 4.4 -2.45) (end 4.4 2.1)
       (stroke (width 0.05) (type solid)) (layer "F.CrtYd"))
-    (fp_line (start 11.25 5.5) (end 8.75 5.5)
+    (fp_line (start 4.4 2.1) (end 1.65 2.1)
       (stroke (width 0.05) (type solid)) (layer "F.CrtYd"))
-    (fp_line (start -2.9 4.5) (end -2.9 -1)
+    (fp_line (start -3.35 -1) (end -3.35 1.6)
       (stroke (width 0.1) (type solid)) (layer "F.Fab"))
-    (fp_line (start -1.9 -2) (end -2.9 -1)
+    (fp_line (start -3.35 1.6) (end 3.35 1.6)
       (stroke (width 0.1) (type solid)) (layer "F.Fab"))
-    (fp_line (start -1.9 -2) (end 10.9 -2)
+    (fp_line (start -1.4 1.65) (end -1.4 2.95)
       (stroke (width 0.1) (type solid)) (layer "F.Fab"))
-    (fp_line (start -0.5 13.5) (end -0.5 4.5)
+    (fp_line (start -1.4 2.95) (end -1.2 3.15)
       (stroke (width 0.1) (type solid)) (layer "F.Fab"))
-    (fp_line (start 4.5 4.5) (end 4.5 13.5)
+    (fp_line (start -1.2 3.15) (end -0.35 3.15)
       (stroke (width 0.1) (type solid)) (layer "F.Fab"))
-    (fp_line (start 4.5 13.5) (end -0.5 13.5)
+    (fp_line (start -0.35 3.15) (end -0.15 2.95)
       (stroke (width 0.1) (type solid)) (layer "F.Fab"))
-    (fp_line (start 10.9 -2) (end 10.9 4.5)
+    (fp_line (start -0.15 2.95) (end -0.1 2.9)
       (stroke (width 0.1) (type solid)) (layer "F.Fab"))
-    (fp_line (start 10.9 4.5) (end -2.9 4.5)
+    (fp_line (start -0.1 2.9) (end -0.1 1.6)
       (stroke (width 0.1) (type solid)) (layer "F.Fab"))
-    (pad "" thru_hole circle (at -2 -1.75) (size 2 2) (drill 1.2) (layers "*.Cu" "*.Mask"))
-    (pad "" thru_hole circle (at -2 4.25) (size 2 2) (drill 1.2) (layers "*.Cu" "*.Mask"))
-    (pad "" thru_hole circle (at 10 -1.75) (size 2 2) (drill 1.2) (layers "*.Cu" "*.Mask"))
-    (pad "" thru_hole circle (at 10 4.25) (size 2 2) (drill 1.2) (layers "*.Cu" "*.Mask"))
-    (pad "1" thru_hole circle (at 0 0) (size 1.7 1.7) (drill 0.9) (layers "*.Cu" "*.Mask")
+    (fp_line (start 3.35 -1) (end -3.35 -1)
+      (stroke (width 0.1) (type solid)) (layer "F.Fab"))
+    (fp_line (start 3.35 1.6) (end 3.35 -1)
+      (stroke (width 0.1) (type solid)) (layer "F.Fab"))
+    (pad "" smd rect (at -3.65 -0.78) (size 1 0.8) (layers "F.Cu" "F.Paste" "F.Mask"))
+    (pad "" smd rect (at -3.65 1.43) (size 1 0.8) (layers "F.Cu" "F.Paste" "F.Mask"))
+    (pad "" np_thru_hole circle (at -1.5 0.33) (size 0.9 0.9) (drill 0.9) (layers "*.Cu" "*.Mask"))
+    (pad "" np_thru_hole circle (at 1.5 0.33) (size 0.9 0.9) (drill 0.9) (layers "*.Cu" "*.Mask"))
+    (pad "" smd rect (at 3.65 -0.78) (size 1 0.8) (layers "F.Cu" "F.Paste" "F.Mask"))
+    (pad "" smd rect (at 3.65 1.43) (size 1 0.8) (layers "F.Cu" "F.Paste" "F.Mask"))
+    (pad "1" smd rect (at -2.25 -1.43) (size 0.7 1.5) (layers "F.Cu" "F.Paste" "F.Mask")
       (net 2 "GND") (pinfunction "A") (pintype "passive"))
-    (pad "2" thru_hole circle (at 4 0) (size 1.7 1.7) (drill 0.9) (layers "*.Cu" "*.Mask")
+    (pad "2" smd rect (at 0.75 -1.43) (size 0.7 1.5) (layers "F.Cu" "F.Paste" "F.Mask")
       (net 19 "/BOOT0_SW") (pinfunction "B") (pintype "passive"))
-    (pad "3" thru_hole circle (at 8 0) (size 1.7 1.7) (drill 0.9) (layers "*.Cu" "*.Mask")
+    (pad "3" smd rect (at 2.25 -1.43) (size 0.7 1.5) (layers "F.Cu" "F.Paste" "F.Mask")
       (net 3 "+3.3V") (pinfunction "C") (pintype "passive"))
-    (model "${KICAD6_3DMODEL_DIR}/Button_Switch_THT.3dshapes/SW_E-Switch_EG1224_SPDT_Angled.wrl"
+    (model "${KICAD6_3DMODEL_DIR}/Button_Switch_SMD.3dshapes/SW_SPDT_PCM12.wrl"
       (offset (xyz 0 0 0))
       (scale (xyz 1 1 1))
